File: Opti-Grow/Opti-Grow.kicad_sch (KiCad schematic)
At the start: 0 parts

Commit message: making the schematic and initial pcb
Parts:
- added J1, J3, J4: Conn_01x03_Pin, Connector_PinHeader_2.00mm:PinHeader_1x03_P2.00mm_Vertical, symbol Connector:Conn_01x03_Pin
- added J5: Conn_01x08_Pin, Connector_PinHeader_2.00mm:PinHeader_1x08_P2.00mm_Vertical, symbol Connector:Conn_01x08_Pin
- added LA1: Lamp, Package_LCC:PLCC-84_29.3x29.3mm_P1.27mm, symbol Device:Lamp
- added M1, M2, M3, M4: Fan, Package_DFN_QFN:VQFN-12-1EP_4x4mm_P0.8mm_EP2.1x2.1mm_ThermalVias, symbol Motor:Fan
- added M5: Motor_DC, Sensor_Audio:Infineon_PG-LLGA-5-2, symbol Motor:Motor_DC
- added PE1, PE2: PeltierElement, symbol Device:PeltierElement
- added U1: ESP32-S3-DEVKITC-1-N8R2, ESP32-S3-DEVKITC-1-N8R2:XCVR_ESP32-S3-DEVKITC-1-N8R2, symbol ESP32-S3-DEVKITC-1-N8R2:ESP32-S3-DEVKITC-1-N8R2
- added U2: (no value), Package_TO_SOT_THT:TO-220-3_Vertical, symbol sensors sympol:LDR
- added U3: DHT22, Sensor:Aosong_DHT11_5.5x12.0_P2.54mm, symbol Sensor:DHT11
- added U4: (no value), Package_SO:SOIC-16_3.9x9.9mm_P1.27mm, symbol sensors sympol:Soil-Moisture
- added U5: (no value), Package_DFN_QFN:WDFN-10-1EP_3x3mm_P0.5mm_EP1.8x2.5mm, symbol sensors sympol:Humidifier
- added U6: (no value), symbol sensors sympol:Grow-light
- added U7: (no value), Package_TO_SOT_SMD:SOT-23, symbol sensors sympol:Power_Supply
- added U8: (no value), Relay_THT:Relay_SPST-NO_Fujitsu_FTR-LYAA005x_FormA_Vertical, symbol sensors sympol:Relay
- added U9: (no value), Package_SON:WSON-8-1EP_6x5mm_P1.27mm_EP3.4x4mm, symbol sensors sympol:StepDown
Connections:
- new net 3V3: J3.3 (Pin_3), J4.3 (Pin_3), U1.J1_1 (3V3), U1.J1_2 (3V3), U2. (VCC), U3.1 (VDD)
- new net DHT22: J3.2 (Pin_2), U1.J1_4 (GPIO4), U3.2 (DATA)
- new net GND: J1.1 (Pin_1), J3.1 (Pin_1), J4.2 (Pin_2), J5.2 (Pin_2), U1.J1_22 (GND), U1.J3_1 (GND), U1.J3_21 (GND), U1.J3_22 (GND), U2. (VCC), U3.4 (GND), U4. (AO), U9. (GND_(OUT))
- new net LDR: J4.1 (Pin_1), U1.J3_5 (GPIO2), U2. (VCC)
- new net VCC: J1.2 (Pin_2), J5.1 (Pin_1), U1.J1_21 (5V0), U4. (AO), U8. (COM_7), U9. (GND_(OUT))
- new net gnd in: U7. (VCC_in), U9. (GND_(OUT))
- new net gnd peltier1: M1.2 (-), M2.2 (-), PE1.1
- new net gnd peltier2: M3.2 (-), M4.2 (-), PE2.1
- new net gnd-grow: U6. (DO)
- new net gnd-heat: LA1.1 (-)
- new net gnd-power: U7. (VCC_in)
- new net gnd-pump: M5.2 (-)
- new net grow: U6. (DO)
- new net growing light: J5.6 (Pin_6), U1.J3_11 (GPIO37), U8. (COM_7)
- new net heat lamp: J5.5 (Pin_5), U1.J3_10 (GPIO38), U8. (COM_7)
- new net humidifier: J5.8 (Pin_8), U1.J3_13 (GPIO35), U8. (COM_7)
- new net peltier 1: J5.4 (Pin_4), U1.J1_14 (GPIO46), U8. (COM_7)
- new net peltier 2: J5.3 (Pin_3), U1.J3_16 (GPIO48), U8. (COM_7)
- new net soil: J1.3 (Pin_3), U1.J3_14 (GPIO0), U4. (AO)
- new net vcc peltier1: M1.1 (+), M2.1 (+), PE1.2
- new net vcc peltier2: M3.1 (+), M4.1 (+), PE2.2
- new net vcc-grow: U6. (DO)
- new net vcc-heat: LA1.2 (+)
- new net vcc-humid: U5. (GND)
- new net vcc-in: U7. (VCC_in)
- new net vcc-power: U7. (VCC_in), U8. (COM_7), U9. (GND_(OUT))
- new net vcc-pump: M5.1 (+)
- new net water pump: J5.7 (Pin_7), U1.J3_12 (GPIO36), U8. (COM_7)
Other:
- note added: "Actuators"
- note added: "Cooling system (Peltiers & Fans)"
- note added: "DHT 22"
- note added: "ESP 32"
- note added: "Heating lamp"
- note added: "Humidifier"
- note added: "LDR"
- note added: "Power Mangement"
- note added: "Power Supply 240W (12V/20A)"
- note added: "Relay 8 channels"
- note added: "Sensors"
- note added: "Sensors Pins"
- note added: "Soil-Moisture"
- note added: "Step-Down 12V --> 5V"
- note added: "UV Grow Light"
- note added: "Water bumb"
- note added: "pins for 3d model of pcb"
